File: electronics/Cell_holder_board/Temperature_sensor.kicad_sch (KiCad schematic)
At the start: 0 parts

Commit message: added temperature sensors and wire pads to "temperature_sensor" sheet
Parts:
- added TH1, TH2, TH3, TH4: Thermistor, symbol Device:Thermistor
- added Temp_1, Temp_2, Temp_3, Temp_4: Prototyping_Pad_Data, BMS_lib:Prototyping_Pad_Data, symbol BMS_lib:Prototyping_Pad_Data
Connections:
- new net: TH1.1, Temp_1.1
- new net: TH3.1, Temp_3.1
- new net: TH4.1, Temp_4.1
- new net: TH2.1, Temp_2.1
- new net GND: TH1.2, TH2.2, TH3.2, TH4.2
Changed lines of the file:
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@@
 (kicad_sch (version 20230121) (generator eeschema)
   (paper "A4")
+  (junction (at 72.39 25.4) (diameter 0) (color 0 0 0 0)
+  )
+  (junction (at 62.23 25.4) (diameter 0) (color 0 0 0 0)
+  )
+  (junction (at 53.34 25.4) (diameter 0) (color 0 0 0 0)
+  )
+  (wire (pts (xy 72.39 25.4) (xy 91.44 25.4))
+    (stroke (width 0) (type default))
+  )
+  (wire (pts (xy 72.39 35.56) (xy 72.39 41.91))
+    (stroke (width 0) (type default))
+  )
+  (wire (pts (xy 34.29 25.4) (xy 53.34 25.4))
+    (stroke (width 0) (type default))
+  )
+  (wire (pts (xy 62.23 22.86) (xy 62.23 25.4))
+    (stroke (width 0) (type default))
+  )
+  (wire (pts (xy 62.23 25.4) (xy 72.39 25.4))
+    (stroke (width 0) (type default))
+  )
+  (wire (pts (xy 53.34 25.4) (xy 62.23 25.4))
+    (stroke (width 0) (type default))
+  )
+  (wire (pts (xy 34.29 35.56) (xy 34.29 41.91))
+    (stroke (width 0) (type default))
+  )
+  (wire (pts (xy 91.44 35.56) (xy 91.44 41.91))
+    (stroke (width 0) (type default))
+  )
+  (wire (pts (xy 53.34 35.56) (xy 53.34 41.91))
+    (stroke (width 0) (type default))
+  )
+  (hierarchical_label "GND" (shape passive) (at 62.23 22.86 90) (fields_autoplaced)
+    (effects (font (size 1.27 1.27)) (justify left))
+  )
+  (symbol (lib_id "Device:Thermistor") (at 34.29 30.48 180) (unit 1)
+    (in_bom yes) (on_board yes) (dnp no) (fields_autoplaced)
+    (property "Reference" "TH1" (at 38.1 29.845 0)
+      (effects (font (size 1.27 1.27)) (justify right))
+    )
+    (property "Value" "Thermistor" (at 38.1 32.385 0)
+      (effects (font (size 1.27 1.27)) (justify right))
+    )
+    (property "Footprint" "" (at 34.29 30.48 0)
+      (effects (font (size 1.27 1.27)) hide)
+    )
+    (property "Datasheet" "~" (at 34.29 30.48 0)
+      (effects (font (size 1.27 1.27)) hide)
+    )
+    (pin "1")
+    (pin "2")
+    (instances
+      (project "Cell_holder_board"
+        (path "/c2697d40-f04f-4888-9ae9-ce0b7f222632/6adc034b-c1df-4fc7-94f9-a847ee71f2c9"
+          (reference "TH1") (unit 1)
+        )
+      )
+    )
+  )
+  (symbol (lib_id "BMS_lib:Prototyping_Pad_Data") (at 72.39 41.91 270) (unit 1)
+    (in_bom yes) (on_board yes) (dnp no)
+    (property "Reference" "Temp_3" (at 72.39 46.99 0)
+      (effects (font (size 1.27 1.27)) (justify left))
+    )
+    (property "Value" "Prototyping_Pad_Data" (at 69.85 43.18 0)
+      (effects (font (size 1.27 1.27)) (justify left))
+    )
+    (property "Footprint" "BMS_lib:Prototyping_Pad_Data" (at 76.2 45.72 0)
+      (effects (font (size 1.27 1.27)) hide)
+    )
+    (property "Datasheet" "" (at 72.39 41.91 0)
+      (effects (font (size 1.27 1.27)) hide)
+    )
+    (pin "1")
+    (instances
+      (project "Cell_holder_board"
+        (path "/c2697d40-f04f-4888-9ae9-ce0b7f222632/6adc034b-c1df-4fc7-94f9-a847ee71f2c9"
+          (reference "Temp_3") (unit 1)
+        )
+      )
+    )
+  )
+  (symbol (lib_id "Device:Thermistor") (at 72.39 30.48 180) (unit 1)
+    (in_bom yes) (on_board yes) (dnp no) (fields_autoplaced)
+    (property "Reference" "TH3" (at 76.2 29.845 0)
+      (effects (font (size 1.27 1.27)) (justify right))
+    )
+    (property "Value" "Thermistor" (at 76.2 32.385 0)
+      (effects (font (size 1.27 1.27)) (justify right))
+    )
+    (property "Footprint" "" (at 72.39 30.48 0)
+      (effects (font (size 1.27 1.27)) hide)
+    )
+    (property "Datasheet" "~" (at 72.39 30.48 0)
+      (effects (font (size 1.27 1.27)) hide)
+    )
+    (pin "1")
+    (pin "2")
+    (instances
+      (project "Cell_holder_board"
+        (path "/c2697d40-f04f-4888-9ae9-ce0b7f222632/6adc034b-c1df-4fc7-94f9-a847ee71f2c9"
+          (reference "TH3") (unit 1)
+        )
+      )
+    )
+  )
+  (symbol (lib_id "Device:Thermistor") (at 91.44 30.48 180) (unit 1)
+    (in_bom yes) (on_board yes) (dnp no) (fields_autoplaced)
+    (property "Reference" "TH4" (at 95.25 29.845 0)
+      (effects (font (size 1.27 1.27)) (justify right))
+    )
+    (property "Value" "Thermistor" (at 95.25 32.385 0)
+      (effects (font (size 1.27 1.27)) (justify right))
+    )
+    (property "Footprint" "" (at 91.44 30.48 0)
+      (effects (font (size 1.27 1.27)) hide)
+    )
+    (property "Datasheet" "~" (at 91.44 30.48 0)
+      (effects (font (size 1.27 1.27)) hide)
+    )
+    (pin "1")
+    (pin "2")
+    (instances
+      (project "Cell_holder_board"
+        (path "/c2697d40-f04f-4888-9ae9-ce0b7f222632/6adc034b-c1df-4fc7-94f9-a847ee71f2c9"
+          (reference "TH4") (unit 1)
+        )
+      )
+    )
+  )
+  (symbol (lib_id "BMS_lib:Prototyping_Pad_Data") (at 91.44 41.91 270) (unit 1)
+    (in_bom yes) (on_board yes) (dnp no)
+    (property "Reference" "Temp_4" (at 91.44 46.99 0)
+      (effects (font (size 1.27 1.27)) (justify left))
+    )
+    (property "Value" "Prototyping_Pad_Data" (at 88.9 43.18 0)
+      (effects (font (size 1.27 1.27)) (justify left))
+    )
+    (property "Footprint" "BMS_lib:Prototyping_Pad_Data" (at 95.25 45.72 0)
+      (effects (font (size 1.27 1.27)) hide)
+    )
+    (property "Datasheet" "" (at 91.44 41.91 0)
+      (effects (font (size 1.27 1.27)) hide)
+    )
+    (pin "1")
+    (instances
+      (project "Cell_holder_board"
+        (path "/c2697d40-f04f-4888-9ae9-ce0b7f222632/6adc034b-c1df-4fc7-94f9-a847ee71f2c9"
+          (reference "Temp_4") (unit 1)
+        )
+      )
+    )
+  )
+  (symbol (lib_id "BMS_lib:Prototyping_Pad_Data") (at 53.34 41.91 270) (unit 1)
+    (in_bom yes) (on_board yes) (dnp no)
+    (property "Reference" "Temp_2" (at 53.34 46.99 0)
+      (effects (font (size 1.27 1.27)) (justify left))
+    )
+    (property "Value" "Prototyping_Pad_Data" (at 50.8 43.18 0)
+      (effects (font (size 1.27 1.27)) (justify left))
+    )
+    (property "Footprint" "BMS_lib:Prototyping_Pad_Data" (at 57.15 45.72 0)
+      (effects (font (size 1.27 1.27)) hide)
+    )
+    (property "Datasheet" "" (at 53.34 41.91 0)
+      (effects (font (size 1.27 1.27)) hide)
+    )
+    (pin "1")
+    (instances
+      (project "Cell_holder_board"
+        (path "/c2697d40-f04f-4888-9ae9-ce0b7f222632/6adc034b-c1df-4fc7-94f9-a847ee71f2c9"
+          (reference "Temp_2") (unit 1)
+        )
+      )
+    )
+  )
+  (symbol (lib_id "Device:Thermistor") (at 53.34 30.48 180) (unit 1)
+    (in_bom yes) (on_board yes) (dnp no) (fields_autoplaced)
+    (property "Reference" "TH2" (at 57.15 29.845 0)
+      (effects (font (size 1.27 1.27)) (justify right))
+    )
+    (property "Value" "Thermistor" (at 57.15 32.385 0)
+      (effects (font (size 1.27 1.27)) (justify right))
+    )
+    (property "Footprint" "" (at 53.34 30.48 0)
+      (effects (font (size 1.27 1.27)) hide)
+    )
+    (property "Datasheet" "~" (at 53.34 30.48 0)
+      (effects (font (size 1.27 1.27)) hide)
+    )
+    (pin "1")
+    (pin "2")
+    (instances
+      (project "Cell_holder_board"
+        (path "/c2697d40-f04f-4888-9ae9-ce0b7f222632/6adc034b-c1df-4fc7-94f9-a847ee71f2c9"
+          (reference "TH2") (unit 1)
+        )
+      )
+    )
+  )
+  (symbol (lib_id "BMS_lib:Prototyping_Pad_Data") (at 34.29 41.91 270) (unit 1)
+    (in_bom yes) (on_board yes) (dnp no)
+    (property "Reference" "Temp_1" (at 34.29 46.99 0)
+      (effects (font (size 1.27 1.27)) (justify left))
+    )
+    (property "Value" "Prototyping_Pad_Data" (at 31.75 43.18 0)
+      (effects (font (size 1.27 1.27)) (justify left))
+    )
+    (property "Footprint" "BMS_lib:Prototyping_Pad_Data" (at 38.1 45.72 0)
+      (effects (font (size 1.27 1.27)) hide)
+    )
+    (property "Datasheet" "" (at 34.29 41.91 0)
+      (effects (font (size 1.27 1.27)) hide)
+    )
+    (pin "1")
+    (instances
+      (project "Cell_holder_board"
+        (path "/c2697d40-f04f-4888-9ae9-ce0b7f222632/6adc034b-c1df-4fc7-94f9-a847ee71f2c9"
+          (reference "Temp_1") (unit 1)
+        )
+      )
+    )
+  )
 )

Commit message: discord session with Johannes and Fabian, Schematic nearly done, all footprints fields filled
Parts:
- removed Temp_1, Temp_2, Temp_3, Temp_4: Prototyping_Pad_Data, BMS_lib:Prototyping_Pad_Data, symbol BMS_lib:Prototyping_Pad_Data
- TH1, TH2, TH3, TH4: footprint (none) -> Resistor_THT:R_Axial_DIN0207_L6.3mm_D2.5mm_P2.54mm_Vertical
Connections:
- net Temp_1: now reaches TH1.1
- net Temp_3: now reaches TH3.1
- net Temp_4: now reaches TH4.1
- net Temp_2: now reaches TH2.1
Changed lines of the file:
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@@
     (stroke (width 0) (type default))
   )
-  (hierarchical_label "GND" (shape passive) (at 62.23 22.86 90) (fields_autoplaced)
-    (effects (font (size 1.27 1.27)) (justify left))
+  (hierarchical_label "Temp_2" (shape bidirectional) (at 53.34 41.91 270) (fields_autoplaced)
+    (effects (font (size 1.27 1.27)) (justify right))
+  )
+  (hierarchical_label "Temp_1" (shape bidirectional) (at 34.29 41.91 270) (fields_autoplaced)
+    (effects (font (size 1.27 1.27)) (justify right))
+  )
+  (hierarchical_label "Temp_4" (shape bidirectional) (at 91.44 41.91 270) (fields_autoplaced)
+    (effects (font (size 1.27 1.27)) (justify right))
+  )
+  (hierarchical_label "Temp_3" (shape bidirectional) (at 72.39 41.91 270) (fields_autoplaced)
+    (effects (font (size 1.27 1.27)) (justify right))
   )
   (symbol (lib_id "Device:Thermistor") (at 34.29 30.48 180) (unit 1)
@@
       (effects (font (size 1.27 1.27)) (justify right))
     )
-    (property "Footprint" "" (at 34.29 30.48 0)
+    (property "Footprint" "Resistor_THT:R_Axial_DIN0207_L6.3mm_D2.5mm_P2.54mm_Vertical" (at 34.29 30.48 0)
       (effects (font (size 1.27 1.27)) hide)
     )
@@
     )
   )
-  (symbol (lib_id "BMS_lib:Prototyping_Pad_Data") (at 72.39 41.91 270) (unit 1)
-    (in_bom yes) (on_board yes) (dnp no)
-    (property "Reference" "Temp_3" (at 72.39 46.99 0)
-      (effects (font (size 1.27 1.27)) (justify left))
-    )
-    (property "Value" "Prototyping_Pad_Data" (at 69.85 43.18 0)
-      (effects (font (size 1.27 1.27)) (justify left))
-    )
-    (property "Footprint" "BMS_lib:Prototyping_Pad_Data" (at 76.2 45.72 0)
-      (effects (font (size 1.27 1.27)) hide)
-    )
-    (property "Datasheet" "" (at 72.39 41.91 0)
-      (effects (font (size 1.27 1.27)) hide)
-    )
-    (pin "1")
-    (instances
-      (project "Cell_holder_board"
-        (path "/c2697d40-f04f-4888-9ae9-ce0b7f222632/6adc034b-c1df-4fc7-94f9-a847ee71f2c9"
-          (reference "Temp_3") (unit 1)
-        )
-      )
-    )
-  )
   (symbol (lib_id "Device:Thermistor") (at 72.39 30.48 180) (unit 1)
     (in_bom yes) (on_board yes) (dnp no) (fields_autoplaced)
@@
       (effects (font (size 1.27 1.27)) (justify right))
     )
-    (property "Footprint" "" (at 72.39 30.48 0)
+    (property "Footprint" "Resistor_THT:R_Axial_DIN0207_L6.3mm_D2.5mm_P2.54mm_Vertical" (at 72.39 30.48 0)
       (effects (font (size 1.27 1.27)) hide)
     )
@@
       (effects (font (size 1.27 1.27)) (justify right))
     )
-    (property "Footprint" "" (at 91.44 30.48 0)
+    (property "Footprint" "Resistor_THT:R_Axial_DIN0207_L6.3mm_D2.5mm_P2.54mm_Vertical" (at 91.44 30.48 0)
       (effects (font (size 1.27 1.27)) hide)
     )
@@
     )
   )
-  (symbol (lib_id "BMS_lib:Prototyping_Pad_Data") (at 91.44 41.91 270) (unit 1)
-    (in_bom yes) (on_board yes) (dnp no)
-    (property "Reference" "Temp_4" (at 91.44 46.99 0)
-      (effects (font (size 1.27 1.27)) (justify left))
-    )
-    (property "Value" "Prototyping_Pad_Data" (at 88.9 43.18 0)
-      (effects (font (size 1.27 1.27)) (justify left))
-    )
-    (property "Footprint" "BMS_lib:Prototyping_Pad_Data" (at 95.25 45.72 0)
+  (symbol (lib_id "power:GND") (at 62.23 22.86 180) (unit 1)
+    (in_bom yes) (on_board yes) (dnp no) (fields_autoplaced)
+    (property "Reference" "#PWR016" (at 62.23 16.51 0)
       (effects (font (size 1.27 1.27)) hide)
     )
-    (property "Datasheet" "" (at 91.44 41.91 0)
+    (property "Value" "GND" (at 62.23 19.05 0)
+      (effects (font (size 1.27 1.27)))
+    )
+    (property "Footprint" "" (at 62.23 22.86 0)
+      (effects (font (size 1.27 1.27)) hide)
+    )
+    (property "Datasheet" "" (at 62.23 22.86 0)
       (effects (font (size 1.27 1.27)) hide)
     )
@@
       (project "Cell_holder_board"
         (path "/c2697d40-f04f-4888-9ae9-ce0b7f222632/6adc034b-c1df-4fc7-94f9-a847ee71f2c9"
-          (reference "Temp_4") (unit 1)
-        )
-      )
-    )
-  )
-  (symbol (lib_id "BMS_lib:Prototyping_Pad_Data") (at 53.34 41.91 270) (unit 1)
-    (in_bom yes) (on_board yes) (dnp no)
-    (property "Reference" "Temp_2" (at 53.34 46.99 0)
-      (effects (font (size 1.27 1.27)) (justify left))
-    )
-    (property "Value" "Prototyping_Pad_Data" (at 50.8 43.18 0)
-      (effects (font (size 1.27 1.27)) (justify left))
-    )
-    (property "Footprint" "BMS_lib:Prototyping_Pad_Data" (at 57.15 45.72 0)
-      (effects (font (size 1.27 1.27)) hide)
-    )
-    (property "Datasheet" "" (at 53.34 41.91 0)
-      (effects (font (size 1.27 1.27)) hide)
-    )
-    (pin "1")
-    (instances
-      (project "Cell_holder_board"
-        (path "/c2697d40-f04f-4888-9ae9-ce0b7f222632/6adc034b-c1df-4fc7-94f9-a847ee71f2c9"
-          (reference "Temp_2") (unit 1)
+          (reference "#PWR016") (unit 1)
         )
       )
@@
       (effects (font (size 1.27 1.27)) (justify right))
     )
-    (property "Footprint" "" (at 53.34 30.48 0)
+    (property "Footprint" "Resistor_THT:R_Axial_DIN0207_L6.3mm_D2.5mm_P2.54mm_Vertical" (at 53.34 30.48 0)
       (effects (font (size 1.27 1.27)) hide)
     )
@@
         )
       )
-    )
-  )
-  (symbol (lib_id "BMS_lib:Prototyping_Pad_Data") (at 34.29 41.91 270) (unit 1)
-    (in_bom yes) (on_board yes) (dnp no)
-    (property "Reference" "Temp_1" (at 34.29 46.99 0)
-      (effects (font (size 1.27 1.27)) (justify left))
-    )
-    (property "Value" "Prototyping_Pad_Data" (at 31.75 43.18 0)
-      (effects (font (size 1.27 1.27)) (justify left))
-    )
-    (property "Footprint" "BMS_lib:Prototyping_Pad_Data" (at 38.1 45.72 0)
-      (effects (font (size 1.27 1.27)) hide)
-    )
-    (property "Datasheet" "" (at 34.29 41.91 0)
-      (effects (font (size 1.27 1.27)) hide)
-    )
-    (pin "1")
-    (instances
-      (project "Cell_holder_board"
-        (path "/c2697d40-f04f-4888-9ae9-ce0b7f222632/6adc034b-c1df-4fc7-94f9-a847ee71f2c9"
-          (reference "Temp_1") (unit 1)
-        )
-      )
