File: electronics/BMS_Project/U_Messung.kicad_sch (KiCad schematic)
At the start: 18 parts, among them U1 LM358, U2 LM358

Commit message: Meeting 28.04.2023 worked on schematic
Connections:
- net U_Bat_1: now also R4.1, U2.1; no longer R1.1, U1.7
- net U_Bat_2: now also R3.1, U2.7; no longer R2.1, U1.1
- net U_Bat_3: now also R2.1, U1.1; no longer R3.1, U2.7
- net U_Bat_4: now also R1.1, U1.7; no longer R4.1, U2.1
- net +12V renamed +BATT
- net BT1_+ renamed BT4_+
- net BT1_-/BT2_+ renamed BT3_+/BT4_-
- net BT2_-/BT3_+ renamed BT2_+/BT3_-
- net BT3_-/BT4_+ renamed BT1_+/BT2_-
Other:
- moved on the sheet: U1C
Changed lines of the file:
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@@
     (stroke (width 0) (type default))
   )
-  (hierarchical_label "BT1_+" (shape bidirectional) (at 127 27.94 0) (fields_autoplaced)
+  (hierarchical_label "BT3_+{slash}BT4_-" (shape bidirectional) (at 127 49.53 0) (fields_autoplaced)
     (effects (font (size 1.27 1.27)) (justify left))
   )
-  (hierarchical_label "U_Bat_3" (shape bidirectional) (at 63.5 110.49 180) (fields_autoplaced)
+  (hierarchical_label "U_Bat_3" (shape bidirectional) (at 63.5 68.58 180) (fields_autoplaced)
     (effects (font (size 1.27 1.27)) (justify right))
   )
-  (hierarchical_label "U_Bat_4" (shape bidirectional) (at 63.5 151.13 180) (fields_autoplaced)
+  (hierarchical_label "U_Bat_4" (shape bidirectional) (at 63.5 30.48 180) (fields_autoplaced)
     (effects (font (size 1.27 1.27)) (justify right))
   )
-  (hierarchical_label "BT1_-{slash}BT2_+" (shape bidirectional) (at 127 49.53 0) (fields_autoplaced)
+  (hierarchical_label "BT2_+{slash}BT3_-" (shape bidirectional) (at 127 87.63 0) (fields_autoplaced)
     (effects (font (size 1.27 1.27)) (justify left))
   )
-  (hierarchical_label "U_Bat_1" (shape bidirectional) (at 63.5 30.48 180) (fields_autoplaced)
+  (hierarchical_label "U_Bat_1" (shape bidirectional) (at 63.5 151.13 180) (fields_autoplaced)
     (effects (font (size 1.27 1.27)) (justify right))
   )
-  (hierarchical_label "BT1_-{slash}BT2_+" (shape bidirectional) (at 127 66.04 0) (fields_autoplaced)
+  (hierarchical_label "U_Bat_2" (shape bidirectional) (at 63.5 110.49 180) (fields_autoplaced)
+    (effects (font (size 1.27 1.27)) (justify right))
+  )
+  (hierarchical_label "BT3_+{slash}BT4_-" (shape bidirectional) (at 127 66.04 0) (fields_autoplaced)
     (effects (font (size 1.27 1.27)) (justify left))
   )
-  (hierarchical_label "U_Bat_2" (shape bidirectional) (at 63.5 68.58 180) (fields_autoplaced)
-    (effects (font (size 1.27 1.27)) (justify right))
-  )
-  (hierarchical_label "BT3_-{slash}BT4_+" (shape bidirectional) (at 127 148.59 0) (fields_autoplaced)
+  (hierarchical_label "BT4_+" (shape bidirectional) (at 127 27.94 0) (fields_autoplaced)
     (effects (font (size 1.27 1.27)) (justify left))
   )
-  (hierarchical_label "BT2_-{slash}BT3_+" (shape bidirectional) (at 127 107.95 0) (fields_autoplaced)
+  (hierarchical_label "BT2_+{slash}BT3_-" (shape bidirectional) (at 127 107.95 0) (fields_autoplaced)
     (effects (font (size 1.27 1.27)) (justify left))
   )
-  (hierarchical_label "BT2_-{slash}BT3_+" (shape bidirectional) (at 127 87.63 0) (fields_autoplaced)
+  (hierarchical_label "BT1_+{slash}BT2_-" (shape bidirectional) (at 127 129.54 0) (fields_autoplaced)
     (effects (font (size 1.27 1.27)) (justify left))
   )
-  (hierarchical_label "BT3_-{slash}BT4_+" (shape bidirectional) (at 127 129.54 0) (fields_autoplaced)
+  (hierarchical_label "BT1_+{slash}BT2_-" (shape bidirectional) (at 127 148.59 0) (fields_autoplaced)
     (effects (font (size 1.27 1.27)) (justify left))
   )
@@
     )
   )
-  (symbol (lib_id "Amplifier_Operational:LM358") (at 66.04 49.53 0) (unit 3)
-    (in_bom yes) (on_board yes) (dnp no) (fields_autoplaced)
-    (property "Reference" "U1" (at 64.77 48.895 0)
-      (effects (font (size 1.27 1.27)) (justify left))
-    )
-    (property "Value" "LM358" (at 64.77 51.435 0)
-      (effects (font (size 1.27 1.27)) (justify left))
-    )
-    (property "Footprint" "Package_LGA:Texas_SIL0008D_MicroSiP-8-1EP_2.8x3mm_P0.65mm_EP1.1x1.9mm" (at 66.04 49.53 0)
-      (effects (font (size 1.27 1.27)) hide)
-    )
-    (property "Datasheet" "http://www.ti.com/lit/ds/symlink/lm2904-n.pdf" (at 66.04 49.53 0)
+  (symbol (lib_id "Amplifier_Operational:LM358") (at 68.58 48.26 0) (unit 3)
+    (in_bom yes) (on_board yes) (dnp no) (fields_autoplaced)
+    (property "Reference" "U1" (at 67.31 47.625 0)
+      (effects (font (size 1.27 1.27)) (justify left))
+    )
+    (property "Value" "LM358" (at 67.31 50.165 0)
+      (effects (font (size 1.27 1.27)) (justify left))
+    )
+    (property "Footprint" "Package_LGA:Texas_SIL0008D_MicroSiP-8-1EP_2.8x3mm_P0.65mm_EP1.1x1.9mm" (at 68.58 48.26 0)
+      (effects (font (size 1.27 1.27)) hide)
+    )
+    (property "Datasheet" "http://www.ti.com/lit/ds/symlink/lm2904-n.pdf" (at 68.58 48.26 0)
       (effects (font (size 1.27 1.27)) hide)
     )
@@
     )
   )
-  (symbol (lib_id "power:+12V") (at 66.04 123.19 0) (unit 1)
-    (in_bom yes) (on_board yes) (dnp no) (fields_autoplaced)
-    (property "Reference" "#PWR03" (at 66.04 127 0)
-      (effects (font (size 1.27 1.27)) hide)
-    )
-    (property "Value" "+12V" (at 66.04 119.38 0)
-      (effects (font (size 1.27 1.27)))
-    )
-    (property "Footprint" "" (at 66.04 123.19 0)
-      (effects (font (size 1.27 1.27)) hide)
-    )
-    (property "Datasheet" "" (at 66.04 123.19 0)
-      (effects (font (size 1.27 1.27)) hide)
-    )
-    (pin "1")
-    (instances
-      (project "BMS_Project"
-        (path "/524e7f14-feb0-4ca2-9425-a347c869bfa6/d8f12774-e346-4091-abf5-b4c43e81469c"
-          (reference "#PWR03") (unit 1)
-        )
-      )
-      (project "Test_Projekt"
-        (path "/d5b120ca-a0f0-4b3f-8fab-ca010d94ac2e"
-          (reference "#PWR06") (unit 1)
-        )
-      )
-    )
-  )
-  (symbol (lib_id "power:+12V") (at 63.5 41.91 0) (unit 1)
-    (in_bom yes) (on_board yes) (dnp no) (fields_autoplaced)
-    (property "Reference" "#PWR01" (at 63.5 45.72 0)
-      (effects (font (size 1.27 1.27)) hide)
-    )
-    (property "Value" "+12V" (at 63.5 38.1 0)
-      (effects (font (size 1.27 1.27)))
-    )
-    (property "Footprint" "" (at 63.5 41.91 0)
-      (effects (font (size 1.27 1.27)) hide)
-    )
-    (property "Datasheet" "" (at 63.5 41.91 0)
-      (effects (font (size 1.27 1.27)) hide)
-    )
-    (pin "1")
-    (instances
-      (project "BMS_Project"
+  (symbol (lib_id "power:+BATT") (at 66.04 40.64 0) (unit 1)
+    (in_bom yes) (on_board yes) (dnp no) (fields_autoplaced)
+    (property "Reference" "#PWR010" (at 66.04 44.45 0)
+      (effects (font (size 1.27 1.27)) hide)
+    )
+    (property "Value" "+BATT" (at 66.04 36.83 0)
+      (effects (font (size 1.27 1.27)))
+    )
+    (property "Footprint" "" (at 66.04 40.64 0)
+      (effects (font (size 1.27 1.27)) hide)
+    )
+    (property "Datasheet" "" (at 66.04 40.64 0)
+      (effects (font (size 1.27 1.27)) hide)
+    )
+    (pin "1")
+    (instances
+      (project "BMS_Project"
+        (path "/524e7f14-feb0-4ca2-9425-a347c869bfa6"
+          (reference "#PWR010") (unit 1)
+        )
         (path "/524e7f14-feb0-4ca2-9425-a347c869bfa6/d8f12774-e346-4091-abf5-b4c43e81469c"
           (reference "#PWR01") (unit 1)
-        )
-      )
-      (project "Test_Projekt"
-        (path "/d5b120ca-a0f0-4b3f-8fab-ca010d94ac2e"
-          (reference "#PWR07") (unit 1)
         )
       )
@@
     )
   )
+  (symbol (lib_id "power:+BATT") (at 66.04 123.19 0) (unit 1)
+    (in_bom yes) (on_board yes) (dnp no) (fields_autoplaced)
+    (property "Reference" "#PWR010" (at 66.04 127 0)
+      (effects (font (size 1.27 1.27)) hide)
+    )
+    (property "Value" "+BATT" (at 66.04 119.38 0)
+      (effects (font (size 1.27 1.27)))
+    )
+    (property "Footprint" "" (at 66.04 123.19 0)
+      (effects (font (size 1.27 1.27)) hide)
+    )
+    (property "Datasheet" "" (at 66.04 123.19 0)
+      (effects (font (size 1.27 1.27)) hide)
+    )
+    (pin "1")
+    (instances
+      (project "BMS_Project"
+        (path "/524e7f14-feb0-4ca2-9425-a347c869bfa6"
+          (reference "#PWR010") (unit 1)
+        )
+        (path "/524e7f14-feb0-4ca2-9425-a347c869bfa6/d8f12774-e346-4091-abf5-b4c43e81469c"
+          (reference "#PWR03") (unit 1)
+        )
+      )
+    )
+  )
   (symbol (lib_id "Device:R") (at 87.63 49.53 90) (unit 1)
     (in_bom yes) (on_board yes) (dnp no) (fields_autoplaced)
@@
     )
   )
-  (symbol (lib_id "power:GND") (at 63.5 57.15 0) (unit 1)
-    (in_bom yes) (on_board yes) (dnp no) (fields_autoplaced)
-    (property "Reference" "#PWR02" (at 63.5 63.5 0)
-      (effects (font (size 1.27 1.27)) hide)
-    )
-    (property "Value" "GND" (at 63.5 62.23 0)
-      (effects (font (size 1.27 1.27)))
-    )
-    (property "Footprint" "" (at 63.5 57.15 0)
-      (effects (font (size 1.27 1.27)) hide)
-    )
-    (property "Datasheet" "" (at 63.5 57.15 0)
-      (effects (font (size 1.27 1.27)) hide)
-    )
+  (symbol (lib_id "power:GND") (at 66.04 55.88 0) (unit 1)
+    (in_bom yes) (on_board yes) (dnp no) (fields_autoplaced)
+    (property "Reference" "#PWR02" (at 66.04 62.23 0)
+      (effects (font (size 1.27 1.27)) hide)
+    )
+    (property "Value" "GND" (at 66.04 60.96 0)
+      (effects (font (size 1.27 1.27)))
+    )
+    (property "Footprint" "" (at 66.04 55.88 0)
+      (effects (font (size 1.27 1.27)) hide)
+    )
+    (property "Datasheet" "" (at 66.04 55.88 0)
+      (effects (font (size 1.27 1.27)) hide)
+    )

Commit message: discord session with Johannes and Fabian, Schematic nearly done, all footprints fields filled
Parts:
- U1, U2: footprint Package_LGA:Texas_SIL0008D_MicroSiP-8-1EP_2.8x3mm_P0.65mm_EP1.1x1.9mm -> Package_DIP:DIP-8_W7.62mm
Changed lines of the file:
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@@
       (effects (font (size 1.27 1.27)))
     )
-    (property "Footprint" "Package_LGA:Texas_SIL0008D_MicroSiP-8-1EP_2.8x3mm_P0.65mm_EP1.1x1.9mm" (at 86.36 110.49 0)
+    (property "Footprint" "Package_DIP:DIP-8_W7.62mm" (at 86.36 110.49 0)
       (effects (font (size 1.27 1.27)) hide)
     )
@@
       (effects (font (size 1.27 1.27)))
     )
-    (property "Footprint" "Package_LGA:Texas_SIL0008D_MicroSiP-8-1EP_2.8x3mm_P0.65mm_EP1.1x1.9mm" (at 86.36 151.13 0)
+    (property "Footprint" "Package_DIP:DIP-8_W7.62mm" (at 86.36 151.13 0)
       (effects (font (size 1.27 1.27)) hide)
     )
@@
       (effects (font (size 1.27 1.27)) (justify left))
     )
-    (property "Footprint" "Package_LGA:Texas_SIL0008D_MicroSiP-8-1EP_2.8x3mm_P0.65mm_EP1.1x1.9mm" (at 68.58 48.26 0)
+    (property "Footprint" "Package_DIP:DIP-8_W7.62mm" (at 68.58 48.26 0)
       (effects (font (size 1.27 1.27)) hide)
     )
@@
       (effects (font (size 1.27 1.27)))
     )
-    (property "Footprint" "Package_LGA:Texas_SIL0008D_MicroSiP-8-1EP_2.8x3mm_P0.65mm_EP1.1x1.9mm" (at 86.36 68.58 0)
+    (property "Footprint" "Package_DIP:DIP-8_W7.62mm" (at 86.36 68.58 0)
       (effects (font (size 1.27 1.27)) hide)
     )
@@
       (effects (font (size 1.27 1.27)))
     )
-    (property "Footprint" "Package_LGA:Texas_SIL0008D_MicroSiP-8-1EP_2.8x3mm_P0.65mm_EP1.1x1.9mm" (at 86.36 30.48 0)
+    (property "Footprint" "Package_DIP:DIP-8_W7.62mm" (at 86.36 30.48 0)
       (effects (font (size 1.27 1.27)) hide)
     )
@@
       (effects (font (size 1.27 1.27)) (justify left))
     )
-    (property "Footprint" "Package_LGA:Texas_SIL0008D_MicroSiP-8-1EP_2.8x3mm_P0.65mm_EP1.1x1.9mm" (at 68.58 130.81 0)
-      (effects (font (size 1.27 1.27)) hide)
-    )
+    (property "Footprint" "Package_DIP:DIP-8_W7.62mm" (at 68.58 130.81 0)
+      (effects (font (size 1.27 1.27)) hide)
+    )

Commit message: Started PCB layout and adjusted schematic to suit the layout needs better
Parts:
- R1, R10, R11, R12, R13, R14, R15, R16, R2, R3, R4, R5, R6, R7, R8, R9: footprint Resistor_THT:R_Axial_DIN0207_L6.3mm_D2.5mm_P10.16mm_Horizontal -> Resistor_SMD:R_0805_2012Metric
Changed lines of the file:
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@@
       (effects (font (size 1.27 1.27)) (justify left))
     )
-    (property "Footprint" "Resistor_THT:R_Axial_DIN0207_L6.3mm_D2.5mm_P10.16mm_Horizontal" (at 98.552 114.3 90)
+    (property "Footprint" "Resistor_SMD:R_0805_2012Metric" (at 98.552 114.3 90)
       (effects (font (size 1.27 1.27)) hide)
     )
@@
       (effects (font (size 1.27 1.27)))
     )
-    (property "Footprint" "Resistor_THT:R_Axial_DIN0207_L6.3mm_D2.5mm_P10.16mm_Horizontal" (at 87.63 171.958 90)
+    (property "Footprint" "Resistor_SMD:R_0805_2012Metric" (at 87.63 171.958 90)
       (effects (font (size 1.27 1.27)) hide)
     )
@@
       (effects (font (size 1.27 1.27)))
     )
-    (property "Footprint" "Resistor_THT:R_Axial_DIN0207_L6.3mm_D2.5mm_P10.16mm_Horizontal" (at 106.68 26.162 90)
+    (property "Footprint" "Resistor_SMD:R_0805_2012Metric" (at 106.68 26.162 90)
       (effects (font (size 1.27 1.27)) hide)
     )
@@
       (effects (font (size 1.27 1.27)) (justify left))
     )
-    (property "Footprint" "Resistor_THT:R_Axial_DIN0207_L6.3mm_D2.5mm_P10.16mm_Horizontal" (at 98.552 154.94 90)
+    (property "Footprint" "Resistor_SMD:R_0805_2012Metric" (at 98.552 154.94 90)
       (effects (font (size 1.27 1.27)) hide)
     )
@@
       (effects (font (size 1.27 1.27)))
     )
-    (property "Footprint" "Resistor_THT:R_Axial_DIN0207_L6.3mm_D2.5mm_P10.16mm_Horizontal" (at 87.63 131.318 90)
+    (property "Footprint" "Resistor_SMD:R_0805_2012Metric" (at 87.63 131.318 90)
       (effects (font (size 1.27 1.27)) hide)
     )
@@
       (effects (font (size 1.27 1.27)))
     )
-    (property "Footprint" "Resistor_THT:R_Axial_DIN0207_L6.3mm_D2.5mm_P10.16mm_Horizontal" (at 106.68 146.812 90)
+    (property "Footprint" "Resistor_SMD:R_0805_2012Metric" (at 106.68 146.812 90)
       (effects (font (size 1.27 1.27)) hide)
     )
@@
       (effects (font (size 1.27 1.27)))
     )
-    (property "Footprint" "Resistor_THT:R_Axial_DIN0207_L6.3mm_D2.5mm_P10.16mm_Horizontal" (at 106.68 127.762 90)
+    (property "Footprint" "Resistor_SMD:R_0805_2012Metric" (at 106.68 127.762 90)
       (effects (font (size 1.27 1.27)) hide)
     )
@@
       (effects (font (size 1.27 1.27)))
     )
-    (property "Footprint" "Resistor_THT:R_Axial_DIN0207_L6.3mm_D2.5mm_P10.16mm_Horizontal" (at 106.68 64.262 90)
+    (property "Footprint" "Resistor_SMD:R_0805_2012Metric" (at 106.68 64.262 90)
       (effects (font (size 1.27 1.27)) hide)
     )
@@
       (effects (font (size 1.27 1.27)) (justify left))
     )
-    (property "Footprint" "Resistor_THT:R_Axial_DIN0207_L6.3mm_D2.5mm_P10.16mm_Horizontal" (at 98.552 72.39 90)
+    (property "Footprint" "Resistor_SMD:R_0805_2012Metric" (at 98.552 72.39 90)
       (effects (font (size 1.27 1.27)) hide)
     )
@@
       (effects (font (size 1.27 1.27)))
     )
-    (property "Footprint" "Resistor_THT:R_Axial_DIN0207_L6.3mm_D2.5mm_P10.16mm_Horizontal" (at 106.68 85.852 90)
+    (property "Footprint" "Resistor_SMD:R_0805_2012Metric" (at 106.68 85.852 90)
       (effects (font (size 1.27 1.27)) hide)
     )
@@
       (effects (font (size 1.27 1.27)))
     )
-    (property "Footprint" "Resistor_THT:R_Axial_DIN0207_L6.3mm_D2.5mm_P10.16mm_Horizontal" (at 87.63 51.308 90)
+    (property "Footprint" "Resistor_SMD:R_0805_2012Metric" (at 87.63 51.308 90)
       (effects (font (size 1.27 1.27)) hide)
     )
@@
       (effects (font (size 1.27 1.27)))
     )
-    (property "Footprint" "Resistor_THT:R_Axial_DIN0207_L6.3mm_D2.5mm_P10.16mm_Horizontal" (at 87.63 89.408 90)
+    (property "Footprint" "Resistor_SMD:R_0805_2012Metric" (at 87.63 89.408 90)
       (effects (font (size 1.27 1.27)) hide)
     )
@@
       (effects (font (size 1.27 1.27)))
     )
-    (property "Footprint" "Resistor_THT:R_Axial_DIN0207_L6.3mm_D2.5mm_P10.16mm_Horizontal" (at 106.68 168.402 90)
+    (property "Footprint" "Resistor_SMD:R_0805_2012Metric" (at 106.68 168.402 90)
       (effects (font (size 1.27 1.27)) hide)
     )
@@
       (effects (font (size 1.27 1.27)) (justify left))
     )
-    (property "Footprint" "Resistor_THT:R_Axial_DIN0207_L6.3mm_D2.5mm_P10.16mm_Horizontal" (at 98.552 34.29 90)
+    (property "Footprint" "Resistor_SMD:R_0805_2012Metric" (at 98.552 34.29 90)
       (effects (font (size 1.27 1.27)) hide)
     )
@@
       (effects (font (size 1.27 1.27)))
     )
-    (property "Footprint" "Resistor_THT:R_Axial_DIN0207_L6.3mm_D2.5mm_P10.16mm_Horizontal" (at 106.68 47.752 90)
+    (property "Footprint" "Resistor_SMD:R_0805_2012Metric" (at 106.68 47.752 90)
       (effects (font (size 1.27 1.27)) hide)
     )
@@
       (effects (font (size 1.27 1.27)))
     )
-    (property "Footprint" "Resistor_THT:R_Axial_DIN0207_L6.3mm_D2.5mm_P10.16mm_Horizontal" (at 106.68 106.172 90)
-      (effects (font (size 1.27 1.27)) hide)
-    )
+    (property "Footprint" "Resistor_SMD:R_0805_2012Metric" (at 106.68 106.172 90)
+      (effects (font (size 1.27 1.27)) hide)
+    )
